File: nRF52832/placa-01.sch (KiCad schematic (older format))
At the start: 0 parts

Commit message: Esquematico
Parts:
- added C1, C11, C12, C2: 12pF, symbol Device:C
- added C10: 1.0µF, symbol Device:C
- added C4, C5, C?: 100nF, symbol Device:C
- added C9: 4.7µ, symbol Device:C
- added L2: 10µH, symbol Device:L
- added L3: 15nH, symbol Device:L
- added U?: myNFR52832, symbol myKicadLib:myNFR52832
- added X1: 32MHz, symbol Device:Crystal
- added X2: 32.768kHz, symbol Device:Crystal
Connections:
- new net: C4.2, U?.1 (DEC1)
- new net: C5.2, U?.13 (VDD)
- new net: C11.1, U?.2 (P0.00/XL1), X2.1
- new net: C10.2, L3.1, U?.46 (DEC4)
- new net: L2.2, U?.47 (DCC)
- new net: C9.2, U?.48 (VDD)
- new net: C12.1, X2.2
- new net: L2.1, L3.2
- new net: C1.1, X1.2
- new net: C2.1, X1.1
- new net GND: C1.2, C10.1, C11.2, C12.2, C2.2, C4.1, C5.1, C9.1, C?.1, U?.45 (VSS)
