File: pager/pager.sch (KiCad schematic (older format))
At the start: 62 parts, among them J1 UART, J2 DC_Adaptor, J3 Battery_Pack, J4 TC2030-CTX-NL, M1 Motor_DC, M2 Motor_DC, SW1 Botão de Reset, U1 nRF52832-QFAA, U2 BQ24075, U3 2450FM07A0029T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

Commit message: Andamento do projeto
Parts:
- removed J2: DC_Adaptor, symbol custom:DC_Adaptor
- added C3: 10nF, Capacitor_SMD:C_0603_1608Metric, symbol Device:C
- added J2: USB_Micro-B, allan:Micro-USB-B_GS-14-2180, symbol custom:USB_Micro-B
- added R19: NF, Resistor_SMD:R_0603_1608Metric, symbol Device:R
- added R20: 0Ω, Resistor_SMD:R_0603_1608Metric, symbol Device:R
- ANT1: footprint (none) -> allan:Antenna_2450AT43B100E
- BZ1: footprint (none) -> allan:BUZZER_PS1240P02BT
- C1, C11, C12, C2, C4, C5, C6, C7, C8: footprint Capacitor_SMD:C_0402_1005Metric -> Capacitor_SMD:C_0603_1608Metric
- C13, C14, C15: footprint (none) -> Capacitor_SMD:C_0603_1608Metric
- C16: footprint (none) -> Capacitor_SMD:CP_Elec_4x5.7
- C17: footprint (none) -> Capacitor_SMD:CP_Elec_4x5.3
- D1, D2, D3, D4, D5, D6: footprint (none) -> LED_SMD:LED_0603_1608Metric
- D7: renamed from D9; value DIODE -> RB520S30T1G; footprint (none) -> allan:DIODE
- D8: renamed from D10; value DIODE -> RB520S30T1G; footprint (none) -> allan:DIODE
- J1: footprint (none) -> Connector_PinHeader_2.00mm:PinHeader_1x03_P2.00mm_Vertical
- J3: footprint (none) -> Connector_JST:JST_PH_B3B-PH-SM4-TB_1x03-1MP_P2.00mm_Vertical
- J4: footprint (none) -> allan:TAG_CONNECT
- L3: footprint Inductor_SMD:L_0402_1005Metric -> Inductor_SMD:L_0603_1608Metric
- M1, M2: footprint (none) -> allan:MOTOR
- R1, R10, R11, R12, R13, R14, R15, R16, R2, R3, R4, R5, R6, R7, R8, R9: footprint (none) -> Resistor_SMD:R_0603_1608Metric
- R17: value 100KΩ -> 4MΩ; footprint (none) -> Resistor_SMD:R_0603_1608Metric
- R18: value 100KΩ -> 10MΩ; footprint (none) -> Resistor_SMD:R_0603_1608Metric
- SW1: value Botão de Reset -> FSMSMTR; footprint (none) -> allan:BUTTON_FSMSMTR
- TR1, TR2, TR3: footprint (none) -> allan:TRANSITOR_MMBT2222AFDICTND
- U1: footprint (none) -> Package_DFN_QFN:QFN-48-1EP_6x6mm_P0.4mm_EP4.6x4.6mm_ThermalVias
- U2: footprint (none) -> allan:BQ24075_RGT0016C_VQFN-16-3x3mm
- U3: footprint (none) -> allan:Balun_2450FM07A0029T
- U4: footprint (none) -> allan:LDO_L78L33CD-TR
Connections:
- net GND: now also C3.1, J2.5 (GND), R19.2
- net IN: now also J2.1 (VCC)
- net MEDIDOR: now also C3.2
- net TERMISTOR: now also R20.2; no longer U2.1 (TS)
- new net: R19.1, R20.1, U2.1 (TS)
- no-connect marks 17 -> 20
Other:
- moved on the sheet: C13, C14, C15, C16, C17, J3, R14, R15, R16, R17, R18, U2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
